Commit message: Inertial Fixes
Fixed center of masses and inertial values to be at the center of the bodies.

File: aster_description/urdf/aster.xacro (robot description, xacro)
@@ -8,8 +8,24 @@
 	</link>
 	<!-->
+	<gazebo>
+		<plugin filename="libgazebo_ros_diff_drive.so" name="differential_drive_controller">
+			<legacyMode>false</legacyMode>
+			<alwaysOn>true</alwaysOn>
+			<updateRate>20</updateRate>
+			<leftJoint>left_wheel_joint</leftJoint>
+			<rightJoint>right_wheel_joint</rightJoint>
+			<wheelSeparation>0.25</wheelSeparation>
+			<wheelDiameter>0.1</wheelDiameter>
+			<torque>0.1</torque>
+			<commandTopic>cmd_vel</commandTopic>
+			<odometryTopic>odom</odometryTopic>
+			<odometryFrame>odom</odometryFrame>
+			<robotBaseFrame>chassis</robotBaseFrame>
+		</plugin>
+	</gazebo>
 	<link name="chassis">
 		<inertial>
-			<mass value="5.0"/>
-			<origin xyz="0.193 0.0 0.080" rpy="0 0 0"/>
+			<mass value="0.906"/>
+			<origin xyz="0.2 0 0.1" rpy="0 0 0"/>
 			<inertia ixx="5.840e-3" ixy="0.0" ixz="1.724e-5" iyy="1.664e-2" iyz="0.0" izz="1.961e-2"/>
 		</inertial>
@@ -45,6 +61,6 @@
 	<link name="right_wheel">
 		<inertial>
-			<mass value="1.0"/>
-			<origin rpy="1.5707 0 0" xyz="0.325 -0.125 0.050"/>
+			<mass value="0.327"/>
+			<origin rpy="0 1.5707 0" xyz="0 0 0"/>
 			<inertia ixx="2.478e-4" ixy="0.0" ixz="0.0" iyy="4.084e-4" iyz="0.0" izz="2.478e-4"/>
 		</inertial>
@@ -64,6 +80,6 @@
 	<link name="left_wheel">
 		<inertial>
-			<mass value="1.0"/>
-			<origin rpy="1.5707 0 0" xyz="0.325 0.125 0.050"/>
+			<mass value="0.327"/>
+			<origin rpy="0 1.5707 0" xyz="0 0 0"/>
 			<inertia ixx="2.478e-4" ixy="0.0" ixz="0.0" iyy="4.084e-4" iyz="0.0" izz="2.478e-4"/>
 		</inertial>

Commit message: Add files via upload

File: aster_description/urdf/aster.xacro (robot description, xacro)
@@ -1,27 +1,7 @@
 <?xml version="1.0"?>
 <robot name="aster" xmlns:xacro="http://www.ros.org/wiki/xacro">
-	<material name="blue">
-		<color rgba="0 0.0 1.0 1.0"/>
-	</material>
-	<!-->
-	<link name="map">
-	</link>
-	<!-->
-	<gazebo>
-		<plugin filename="libgazebo_ros_diff_drive.so" name="differential_drive_controller">
-			<legacyMode>false</legacyMode>
-			<alwaysOn>true</alwaysOn>
-			<updateRate>20</updateRate>
-			<leftJoint>left_wheel_joint</leftJoint>
-			<rightJoint>right_wheel_joint</rightJoint>
-			<wheelSeparation>0.25</wheelSeparation>
-			<wheelDiameter>0.1</wheelDiameter>
-			<torque>0.1</torque>
-			<commandTopic>cmd_vel</commandTopic>
-			<odometryTopic>odom</odometryTopic>
-			<odometryFrame>odom</odometryFrame>
-			<robotBaseFrame>chassis</robotBaseFrame>
-		</plugin>
-	</gazebo>
+	<xacro:include filename="$(find aster_description)/urdf/materials.xacro"/>
+	<xacro:include filename="$(find aster_description)/urdf/aster.gazebo"/>
+	<xacro:include filename="$(find aster_description)/urdf/macros.xacro"/>
 	<link name="chassis">
 		<inertial>
@@ -59,63 +39,7 @@
 		</visual>
 	</link>
-	<link name="right_wheel">
-		<inertial>
-			<mass value="0.327"/>
-			<origin rpy="0 1.5707 0" xyz="0 0 0"/>
-			<inertia ixx="2.478e-4" ixy="0.0" ixz="0.0" iyy="4.084e-4" iyz="0.0" izz="2.478e-4"/>
-		</inertial>
-		<visual name="visual">
-			<origin rpy="1.5707 0 0" xyz="0 0 0"/>
-			<geometry>
-				<cylinder length="0.04" radius="0.05"/>
-			</geometry>
-		</visual>
-		<collision name="collision">
-			<origin rpy="1.5707 0 0" xyz="0 0 0"/>
-			<geometry>
-				<cylinder length="0.04" radius="0.05"/>
-			</geometry>
-		</collision>
-	</link>
-	<link name="left_wheel">
-		<inertial>
-			<mass value="0.327"/>
-			<origin rpy="0 1.5707 0" xyz="0 0 0"/>
-			<inertia ixx="2.478e-4" ixy="0.0" ixz="0.0" iyy="4.084e-4" iyz="0.0" izz="2.478e-4"/>
-		</inertial>
-		<visual name="visual">
-			<origin rpy="1.5707 0 0" xyz="0 0 0"/>
-			<geometry>
-				<cylinder length="0.04" radius="0.05"/>
-			</geometry>
-		</visual>
-		<collision name="collision">
-			<origin rpy="1.5707 0 0" xyz="0 0 0"/>
-			<geometry>
-				<cylinder length="0.04" radius=	"0.05"/>
-			</geometry>
-		</collision>
-	</link>
-	<!-->
-	<joint name="dummy_joint" type="floating">
-		<parent link="map"/>
-		<child link="chassis"/>
-	</joint>
-	<!-->
-	<joint name="right_wheel_joint" type="continuous">
-		<parent link="chassis"/>
-		<child link="right_wheel"/>
-		<axis xyz="0 1 0" rpy="0 0 0"/>
-		<origin xyz="0.325 -0.125 0.050"/>
-		<joint_properties damping="1.0" friction="1.0"/>
-		<limit effort="1000" velocity="1000"/>
-	</joint>
-	<joint name="left_wheel_joint" type="continuous">
-		<parent link="chassis"/>
-		<child link="left_wheel"/>
-		<axis xyz="0 1 0" rpy="0 0 0"/>
-		<origin xyz="0.325 0.125 0.050"/>
-		<joint_properties damping="1.0" friction="1.0"/>
-		<limit effort="1000" velocity="1000"/>
-	</joint>
+	<xacro:wheel name="right_wheel" />
+	<xacro:wheel_joint name="right_wheel_joint" child="right_wheel" origin_xyz="0.325 -0.125 0.050" />
+	<xacro:wheel name="left_wheel" />
+	<xacro:wheel_joint name="left_wheel_joint" child="left_wheel" origin_xyz="0.325 0.125 0.050" />
 </robot>

Commit message: Added Laser, colors to Aster
Added laser Plugin to visualize laser data.
Added gazebo colours to colorize robot during simulation.

File: aster_description/urdf/aster.xacro (robot description, xacro)
@@ -24,5 +24,5 @@
 			<material name="blue"/>
 		</collision>
-		<visual name="visual">
+		<visual>
 			<origin xyz="0.2 0 0.1" rpy="0 0 0"/>
 			<geometry>
@@ -39,4 +39,28 @@
 		</visual>
 	</link>
+	<link name="sensor_laser">
+		<inertial>
+			<origin xyz="0 0 0" rpy="0 0 0"/>
+			<mass value="0.052"/>
+			<inertia ixx="1.076e-5" ixy="0.0" ixz="0.0" iyy="1.076e-5" iyz="0.0" izz="1.614e-5"/>
+		</inertial>
+		<visual name="visual_laser_sensor">
+			<origin xyz="0 0 0" rpy="0 0 0"/>
+			<geometry>
+				<cylinder radius="0.025" length="0.025"/>
+			</geometry>
+		</visual>
+		<collision name="collisison_laser_sensor">
+			<origin xyz="0 0 0" rpy="0 0 0"/>
+			<geometry>
+				<cylinder radius="0.025" length="0.025"/>
+			</geometry>
+		</collision>
+	</link>
+	<joint name="joint_sensor_laser" type="fixed">
+		<parent link="chassis"/>
+		<child link="sensor_laser"/>
+		<origin xyz="0.358 0.0 0.168" rpy="0 0 0"  />
+	</joint>
 	<xacro:wheel name="right_wheel" />
 	<xacro:wheel_joint name="right_wheel_joint" child="right_wheel" origin_xyz="0.325 -0.125 0.050" />

File: aster_description/urdf/macros.xacro (robot description, xacro)
@@ -8,5 +8,5 @@
 			<inertia ixx="2.478e-4" ixy="0.0" ixz="0.0" iyy="4.084e-4" iyz="0.0" izz="2.478e-4"/>
 		</inertial>
-		<visual name="${name}_visual">
+		<visual>
 			<origin rpy="1.5707 0 0" xyz="0 0 0"/>
 			<geometry>
@@ -14,5 +14,5 @@
 			</geometry>
 		</visual>
-		<collision name="${name}_collision">
+		<collision name="$collision_{name">
 			<origin rpy="1.5707 0 0" xyz="0 0 0"/>
 			<geometry>

File: aster_description/urdf/materials.xacro (robot description, xacro)
@@ -4,3 +4,15 @@
 		<color rgba="0 0.0 1.0 1.0"/>
 	</material>
+	<gazebo reference="chassis">
+		<material>Gazebo/Orange</material>
+	</gazebo>
+	<gazebo reference="right_wheel">
+		<material>Gazebo/Blue</material>
+	</gazebo>
+	<gazebo reference="left_wheel">
+		<material>Gazebo/Blue</material>
+	</gazebo>
+	<gazebo reference="visual_laser_sensor">
+		<material>Gazebo/White</material>
+	</gazebo>
 </robot>
